Commit message: feat(v2.4): complete autonomous navigation upgrade
- Deploy YOLOv8n V2.4 10-class visual perception with directional sign parsing
- Implement real-time Camera-LiDAR TTC range-rate tracking and proactive yielding
- Enhance realistic facility world: eliminate doorway bottlenecks, align signs
- Optimize system CPU by ~32-42% via frame-skipping, JPEG caching, node pruning
- Add real-time [FUSED] 3D perception dashboard and SQLite WAL concurrency
- Complete comprehensive 10-mission automated validation and benchmark suite

File: ros2_ws/src/autonomous_robot_description/urdf/camera.xacro (robot description, xacro)
@@ -24,5 +24,5 @@
     <parent link="base_link"/>
     <child link="camera_link"/>
-    <origin xyz="0.22 0 0.12" rpy="0 0 0"/>
+    <origin xyz="0.22 0 0.35" rpy="0 -0.05 0"/>
   </joint>
   <!-- Camera Optical Link (Standard ROS / OpenCV frame: Z forward, X right, Y down) -->
@@ -43,5 +43,5 @@
       <camera>
         <camera_info_topic>/camera/camera_info</camera_info_topic>
-        <horizontal_fov>1.089</horizontal_fov>
+        <horizontal_fov>1.15</horizontal_fov>
         <image>
           <width>640</width>
